File: Hub_Board_PCB/central_hub/MCU_Sheet.kicad_sch (KiCad schematic)
At the start: 40 parts, among them SW2 SW_Push, U1 R7FA4M1AB3CFM, Y1 16MHz

Commit message: Schematic changes before sending to kim
Parts:
- removed R4: 5.1k, Resistor_SMD:R_0603_1608Metric, symbol Device:R
- R3: value 5.1k -> 10k
Connections:
- net GND: now also R3.2
- net A4 renamed SDA_Accel
- net A5 renamed SCL_Accel
Changed lines of the file:
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@@
   (junction (at 115.57 72.39) (diameter 0) (color 0 0 0 0)
   )
-  (junction (at 224.79 64.77) (diameter 0) (color 0 0 0 0)
-  )
   (junction (at 82.55 85.09) (diameter 0) (color 0 0 0 0)
   )
@@
   )
   (junction (at 90.17 59.69) (diameter 0) (color 0 0 0 0)
-  )
-  (junction (at 220.98 62.23) (diameter 0) (color 0 0 0 0)
   )
   (junction (at 118.11 107.95) (diameter 0) (color 0 0 0 0)
@@
     (stroke (width 0) (type default))
   )
-  (wire (pts (xy 190.5 62.23) (xy 220.98 62.23))
-    (stroke (width 0) (type default))
-  )
   (wire (pts (xy 190.5 77.47) (xy 228.6 77.47))
     (stroke (width 0) (type default))
@@
     (stroke (width 0) (type default))
   )
-  (wire (pts (xy 224.79 55.88) (xy 224.79 64.77))
-    (stroke (width 0) (type default))
-  )
   (wire (pts (xy 115.57 69.85) (xy 115.57 72.39))
     (stroke (width 0) (type default))
@@
     (stroke (width 0) (type default))
   )
-  (wire (pts (xy 91.44 140.97) (xy 91.44 142.24))
-    (stroke (width 0) (type default))
-  )
   (wire (pts (xy 73.66 88.9) (xy 73.66 87.63))
     (stroke (width 0) (type default))
@@
     (stroke (width 0) (type default))
   )
-  (wire (pts (xy 220.98 62.23) (xy 228.6 62.23))
+  (wire (pts (xy 190.5 62.23) (xy 228.6 62.23))
     (stroke (width 0) (type default))
   )
@@
     (stroke (width 0) (type default))
   )
-  (wire (pts (xy 91.44 149.86) (xy 91.44 151.13))
+  (wire (pts (xy 91.44 140.97) (xy 91.44 146.05))
     (stroke (width 0) (type default))
   )
@@
     (stroke (width 0) (type default))
   )
-  (wire (pts (xy 224.79 64.77) (xy 228.6 64.77))
+  (wire (pts (xy 190.5 64.77) (xy 228.6 64.77))
     (stroke (width 0) (type default))
   )
@@
     (stroke (width 0) (type default))
   )
-  (wire (pts (xy 190.5 64.77) (xy 224.79 64.77))
-    (stroke (width 0) (type default))
-  )
   (wire (pts (xy 93.98 92.71) (xy 119.38 92.71))
     (stroke (width 0) (type default))
@@
   )
   (wire (pts (xy 72.39 59.69) (xy 76.2 59.69))
-    (stroke (width 0) (type default))
-  )
-  (wire (pts (xy 220.98 55.88) (xy 220.98 62.23))
     (stroke (width 0) (type default))
   )
@@
     )
   )
-  (global_label "A4" (shape input) (at 224.79 55.88 90) (fields_autoplaced)
-    (effects (font (size 1.27 1.27)) (justify left))
-    (property "Intersheetrefs" "${INTERSHEET_REFS}" (at 224.79 50.5967 90)
-      (effects (font (size 1.27 1.27)) (justify left) hide)
-    )
-  )
   (global_label "SCL_Accel" (shape input) (at 228.6 62.23 0) (fields_autoplaced)
     (effects (font (size 1.27 1.27)) (justify left))
@@
     (effects (font (size 1.27 1.27)) (justify left))
     (property "Intersheetrefs" "${INTERSHEET_REFS}" (at 216.1033 39.37 0)
-      (effects (font (size 1.27 1.27)) (justify left) hide)
-    )
-  )
-  (global_label "A5" (shape input) (at 220.98 55.88 90) (fields_autoplaced)
-    (effects (font (size 1.27 1.27)) (justify left))
-    (property "Intersheetrefs" "${INTERSHEET_REFS}" (at 220.98 50.5967 90)
       (effects (font (size 1.27 1.27)) (justify left) hide)
     )
@@
     )
   )
-  (symbol (lib_id "power:GND") (at 91.44 151.13 0) (unit 1)
-    (in_bom yes) (on_board yes) (dnp no)
-    (property "Reference" "#PWR017" (at 91.44 157.48 0)
-      (effects (font (size 1.27 1.27)) hide)
-    )
-    (property "Value" "GND" (at 91.44 156.21 0)
-      (effects (font (size 1.27 1.27)))
-    )
-    (property "Footprint" "" (at 91.44 151.13 0)
-      (effects (font (size 1.27 1.27)) hide)
-    )
-    (property "Datasheet" "" (at 91.44 151.13 0)
+  (symbol (lib_id "power:GND") (at 91.44 146.05 0) (unit 1)
+    (in_bom yes) (on_board yes) (dnp no)
+    (property "Reference" "#PWR017" (at 91.44 152.4 0)
+      (effects (font (size 1.27 1.27)) hide)
+    )
+    (property "Value" "GND" (at 91.44 151.13 0)
+      (effects (font (size 1.27 1.27)))
+    )
+    (property "Footprint" "" (at 91.44 146.05 0)
+      (effects (font (size 1.27 1.27)) hide)
+    )
+    (property "Datasheet" "" (at 91.44 146.05 0)
       (effects (font (size 1.27 1.27)) hide)
     )
@@
       (effects (font (size 1.27 1.27)) (justify left))
     )
-    (property "Value" "5.1k" (at 93.98 138.43 0)
+    (property "Value" "10k" (at 93.98 138.43 0)
       (effects (font (size 1.27 1.27)) (justify left))
     )
@@
         )
       )
-    )
-  )
-  (symbol (lib_id "Device:R") (at 91.44 146.05 0) (unit 1)
-    (in_bom yes) (on_board yes) (dnp no) (fields_autoplaced)
-    (property "Reference" "R4" (at 93.98 144.78 0)
-      (effects (font (size 1.27 1.27)) (justify left))
-    )
-    (property "Value" "5.1k" (at 93.98 147.32 0)
-      (effects (font (size 1.27 1.27)) (justify left))
-    )
-    (property "Footprint" "Resistor_SMD:R_0603_1608Metric" (at 89.662 146.05 90)
-      (effects (font (size 1.27 1.27)) hide)
-    )
-    (property "Datasheet" "~" (at 91.44 146.05 0)
-      (effects (font (size 1.27 1.27)) hide)
-    )
-    (pin "1")
-    (pin "2")
-    (instances
-      (project "central_hub"
-        (path "/0d9ec66e-0fbf-4d12-9b83-adf78971a00b"
-          (reference "R4") (unit 1)
-        )
-        (path "/0d9ec66e-0fbf-4d12-9b83-adf78971a00b/4fb60496-ee10-4e45-a75e-a49c2c8afc68"
-          (reference "R7") (unit 1)
-        )
-      )
