File: Hub_Board_PCB/central_hub/MCU_Sheet.kicad_sch (KiCad schematic)
At the start: 39 parts, among them SW2 SW_Push, U1 R7FA4M1AB3CFM, Y1 16MHz

Commit message: Central hub layout first draft (+ some changes to motor driver)
Parts:
- removed SW2: SW_Push, Button_Switch_SMD:SW_Push_1P1T_NO_6x6mm_H9.5mm, symbol Switch:SW_Push
- removed TP1, TP7: TestPoint, TestPoint:TestPoint_Pad_D1.0mm, symbol Connector:TestPoint
Changed lines of the file:
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@@
   (junction (at 118.11 105.41) (diameter 0) (color 0 0 0 0)
-  )
-  (junction (at 39.37 44.45) (diameter 0) (color 0 0 0 0)
-  )
-  (junction (at 97.79 69.85) (diameter 0) (color 0 0 0 0)
   )
   (junction (at 91.44 132.08) (diameter 0) (color 0 0 0 0)
@@
     (stroke (width 0) (type default))
   )
-  (wire (pts (xy 97.79 69.85) (xy 115.57 69.85))
-    (stroke (width 0) (type default))
-  )
   (wire (pts (xy 76.2 80.01) (xy 78.74 80.01))
     (stroke (width 0) (type default))
@@
     (stroke (width 0) (type default))
   )
-  (wire (pts (xy 58.42 175.26) (xy 58.42 176.53))
-    (stroke (width 0) (type default))
-  )
   (wire (pts (xy 115.57 72.39) (xy 115.57 74.93))
     (stroke (width 0) (type default))
@@
     (stroke (width 0) (type default))
   )
-  (wire (pts (xy 90.17 69.85) (xy 97.79 69.85))
+  (wire (pts (xy 90.17 69.85) (xy 115.57 69.85))
     (stroke (width 0) (type default))
   )
@@
     (stroke (width 0) (type default))
   )
-  (wire (pts (xy 25.4 44.45) (xy 24.13 44.45))
-    (stroke (width 0) (type default))
-  )
   (wire (pts (xy 82.55 96.52) (xy 82.55 97.79))
     (stroke (width 0) (type default))
@@
     (stroke (width 0) (type default))
   )
-  (wire (pts (xy 24.13 44.45) (xy 24.13 45.72))
-    (stroke (width 0) (type default))
-  )
   (wire (pts (xy 190.5 64.77) (xy 228.6 64.77))
-    (stroke (width 0) (type default))
-  )
-  (wire (pts (xy 39.37 44.45) (xy 35.56 44.45))
     (stroke (width 0) (type default))
   )
@@
     )
   )
-  (symbol (lib_id "power:GND") (at 24.13 45.72 0) (unit 1)
-    (in_bom yes) (on_board yes) (dnp no) (fields_autoplaced)
-    (property "Reference" "#PWR043" (at 24.13 52.07 0)
-      (effects (font (size 1.27 1.27)) hide)
-    )
-    (property "Value" "GND" (at 24.13 50.8 0)
-      (effects (font (size 1.27 1.27)))
-    )
-    (property "Footprint" "" (at 24.13 45.72 0)
-      (effects (font (size 1.27 1.27)) hide)
-    )
-    (property "Datasheet" "" (at 24.13 45.72 0)
-      (effects (font (size 1.27 1.27)) hide)
-    )
-    (pin "1")
-    (instances
-      (project "central_hub"
-        (path "/0d9ec66e-0fbf-4d12-9b83-adf78971a00b"
-          (reference "#PWR043") (unit 1)
-        )
-        (path "/0d9ec66e-0fbf-4d12-9b83-adf78971a00b/4fb60496-ee10-4e45-a75e-a49c2c8afc68"
-          (reference "#PWR01") (unit 1)
-        )
-      )
-    )
-  )
   (symbol (lib_id "Device:R") (at 120.65 181.61 0) (unit 1)
     (in_bom yes) (on_board yes) (dnp no) (fields_autoplaced)
@@
         (path "/0d9ec66e-0fbf-4d12-9b83-adf78971a00b/4fb60496-ee10-4e45-a75e-a49c2c8afc68"
           (reference "#PWR019") (unit 1)
-        )
-      )
-    )
-  )
-  (symbol (lib_id "VIN:VIN") (at 52.07 168.91 0) (unit 1)
-    (in_bom no) (on_board no) (dnp no) (fields_autoplaced)
-    (property "Reference" "#PWR066" (at 58.42 177.8 0) (do_not_autoplace)
-      (effects (font (size 1.27 1.27)) hide)
-    )
-    (property "Value" "VIN" (at 58.42 170.18 0)
-      (effects (font (size 1.27 1.27)))
-    )
-    (property "Footprint" "" (at 52.07 168.91 0)
-      (effects (font (size 1.27 1.27)) hide)
-    )
-    (property "Datasheet" "" (at 52.07 168.91 0)
-      (effects (font (size 1.27 1.27)) hide)
-    )
-    (pin "1")
-    (instances
-      (project "central_hub"
-        (path "/0d9ec66e-0fbf-4d12-9b83-adf78971a00b"
-          (reference "#PWR066") (unit 1)
-        )
-        (path "/0d9ec66e-0fbf-4d12-9b83-adf78971a00b/4fb60496-ee10-4e45-a75e-a49c2c8afc68"
-          (reference "#PWR06") (unit 1)
         )
       )
@@
     )
   )
-  (symbol (lib_id "Connector:TestPoint") (at 97.79 69.85 0) (unit 1)
-    (in_bom yes) (on_board yes) (dnp no)
-    (property "Reference" "TP1" (at 99.06 67.31 0)
-      (effects (font (size 1.27 1.27)) (justify left))
-    )
-    (property "Value" "TestPoint" (at 100.33 67.818 0)
-      (effects (font (size 1.27 1.27)) (justify left) hide)
-    )
-    (property "Footprint" "TestPoint:TestPoint_Pad_D1.0mm" (at 102.87 69.85 0)
-      (effects (font (size 1.27 1.27)) hide)
-    )
-    (property "Datasheet" "~" (at 102.87 69.85 0)
-      (effects (font (size 1.27 1.27)) hide)
-    )
-    (pin "1")
-    (instances
-      (project "central_hub"
-        (path "/0d9ec66e-0fbf-4d12-9b83-adf78971a00b"
-          (reference "TP1") (unit 1)
-        )
-        (path "/0d9ec66e-0fbf-4d12-9b83-adf78971a00b/4fb60496-ee10-4e45-a75e-a49c2c8afc68"
-          (reference "TP6") (unit 1)
-        )
-      )
-    )
-  )
   (symbol (lib_id "Device:LED") (at 134.62 171.45 90) (unit 1)
     (in_bom yes) (on_board yes) (dnp no)
@@
     )
   )
-  (symbol (lib_id "Connector:TestPoint") (at 58.42 176.53 180) (unit 1)
-    (in_bom yes) (on_board yes) (dnp no)
-    (property "Reference" "TP7" (at 60.96 182.88 0)
-      (effects (font (size 1.27 1.27)) (justify left))
-    )
-    (property "Value" "TestPoint" (at 55.88 178.562 0)
-      (effects (font (size 1.27 1.27)) (justify left) hide)
-    )
-    (property "Footprint" "TestPoint:TestPoint_Pad_D1.0mm" (at 53.34 176.53 0)
-      (effects (font (size 1.27 1.27)) hide)
-    )
-    (property "Datasheet" "~" (at 53.34 176.53 0)
-      (effects (font (size 1.27 1.27)) hide)
-    )
-    (pin "1")
-    (instances
-      (project "central_hub"
-        (path "/0d9ec66e-0fbf-4d12-9b83-adf78971a00b"
-          (reference "TP7") (unit 1)
-        )
-        (path "/0d9ec66e-0fbf-4d12-9b83-adf78971a00b/4fb60496-ee10-4e45-a75e-a49c2c8afc68"
-          (reference "TP1") (unit 1)
-        )
-      )
-    )
-  )
   (symbol (lib_id "Device:C") (at 80.01 52.07 90) (unit 1)
     (in_bom yes) (on_board yes) (dnp no) (fields_autoplaced)
@@
         )
       )
-    )
-  )
-  (symbol (lib_id "Switch:SW_Push") (at 30.48 44.45 0) (unit 1)
-    (in_bom yes) (on_board yes) (dnp no) (fields_autoplaced)
-    (property "Reference" "SW2" (at 30.48 36.83 0)
-      (effects (font (size 1.27 1.27)))
-    )
-    (property "Value" "SW_Push" (at 30.48 39.37 0)
-      (effects (font (size 1.27 1.27)))
-    )
-    (property "Footprint" "Button_Switch_SMD:SW_Push_1P1T_NO_6x6mm_H9.5mm" (at 30.48 39.37 0)
-      (effects (font (size 1.27 1.27)) hide)
-    )
-    (property "Datasheet" "~" (at 30.48 39.37 0)
-      (effects (font (size 1.27 1.27)) hide)
-    )
-    (pin "1")
-    (pin "2")
-    (instances
-      (project "central_hub"
-        (path "/0d9ec66e-0fbf-4d12-9b83-adf78971a00b"
-          (reference "SW2") (unit 1)
-        )
-        (path "/0d9ec66e-0fbf-4d12-9b83-adf78971a00b/4fb60496-ee10-4e45-a75e-a49c2c8afc68"
-          (reference "SW1") (unit 1)
-        )
-      )

Commit message: Meeting layout updates
Parts:
- added R7 (x3): 0, Resistor_SMD:R_0402_1005Metric, symbol Device:R
Connections:
- net D10: now also R7.1; no longer U1.37 (GTIOC3B/P112)
- net D11: now also R7.1; no longer U1.34 (CTX0/TDO/SWO/GTIOC1A/P109)
- net D13: now also R7.1; no longer U1.36 (GTIOC3A/P111)
- new net: R7.2, U1.34 (CTX0/TDO/SWO/GTIOC1A/P109)
- new net: R7.2, U1.36 (GTIOC3A/P111)
- new net: R7.2, U1.37 (GTIOC3B/P112)
Changed lines of the file:
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@@
-    (stroke (width 0) (type default))
-  )
-  (wire (pts (xy 190.5 87.63) (xy 208.28 87.63))
     (stroke (width 0) (type default))
   )
@@
     (stroke (width 0) (type default))
   )
+  (wire (pts (xy 198.12 90.17) (xy 215.9 90.17))
+    (stroke (width 0) (type default))
+  )
   (wire (pts (xy 24.13 181.61) (xy 24.13 182.88))
     (stroke (width 0) (type default))
@@
     (stroke (width 0) (type default))
   )
-  (wire (pts (xy 190.5 90.17) (xy 208.28 90.17))
-    (stroke (width 0) (type default))
-  )
   (wire (pts (xy 115.57 72.39) (xy 115.57 74.93))
     (stroke (width 0) (type default))
@@
     (stroke (width 0) (type default))
   )
+  (wire (pts (xy 198.12 92.71) (xy 215.9 92.71))
+    (stroke (width 0) (type default))
+  )
   (wire (pts (xy 83.82 69.85) (xy 90.17 69.85))
     (stroke (width 0) (type default))
@@
     (stroke (width 0) (type default))
   )
+  (wire (pts (xy 190.5 87.63) (xy 215.9 87.63))
+    (stroke (width 0) (type default))
+  )
   (wire (pts (xy 73.66 88.9) (xy 73.66 87.63))
     (stroke (width 0) (type default))
@@
     (stroke (width 0) (type default))
   )
-  (wire (pts (xy 190.5 85.09) (xy 208.28 85.09))
-    (stroke (width 0) (type default))
-  )
   (wire (pts (xy 190.5 128.27) (xy 233.68 128.27))
     (stroke (width 0) (type default))
@@
     (stroke (width 0) (type default))
   )
-  (wire (pts (xy 190.5 92.71) (xy 208.28 92.71))
-    (stroke (width 0) (type default))
-  )
   (wire (pts (xy 165.1 168.91) (xy 165.1 166.37))
     (stroke (width 0) (type default))
@@
   )
   (wire (pts (xy 106.68 123.19) (xy 119.38 123.19))
+    (stroke (width 0) (type default))
+  )
+  (wire (pts (xy 198.12 85.09) (xy 215.9 85.09))
     (stroke (width 0) (type default))
   )
@@
     (effects (font (size 1.27 1.27)) (justify left bottom))
   )
-  (label "P109_SCI9_TXD" (at 191.77 85.09 0) (fields_autoplaced)
+  (label "P109_SCI9_TXD" (at 201.93 85.09 0) (fields_autoplaced)
     (effects (font (size 1.27 1.27)) (justify left bottom))
   )
@@
     (effects (font (size 1.27 1.27)) (justify left bottom))
   )
-  (label "P111_GPT3_A" (at 191.77 90.17 0) (fields_autoplaced)
+  (label "P111_GPT3_A" (at 201.93 90.17 0) (fields_autoplaced)
     (effects (font (size 1.27 1.27)) (justify left bottom))
   )
@@
     (effects (font (size 1.27 1.27)) (justify left bottom))
   )
-  (label "P112_GPT3_B" (at 191.77 92.71 0) (fields_autoplaced)
+  (label "P112_GPT3_B" (at 201.93 92.71 0) (fields_autoplaced)
     (effects (font (size 1.27 1.27)) (justify left bottom))
   )
@@
     (effects (font (size 1.27 1.27)) (justify left bottom))
   )
-  (label "P110_SCI9_RXD" (at 191.77 87.63 0) (fields_autoplaced)
+  (label "P110_SCI9_RXD" (at 201.93 87.63 0) (fields_autoplaced)
     (effects (font (size 1.27 1.27)) (justify left bottom))
   )
@@
     )
   )
-  (global_label "D11" (shape input) (at 208.28 85.09 0) (fields_autoplaced)
+  (global_label "D11" (shape input) (at 215.9 85.09 0) (fields_autoplaced)
     (effects (font (size 1.27 1.27)) (justify left))
-    (property "Intersheetrefs" "${INTERSHEET_REFS}" (at 214.9542 85.09 0)
+    (property "Intersheetrefs" "${INTERSHEET_REFS}" (at 222.5742 85.09 0)
       (effects (font (size 1.27 1.27)) (justify left) hide)
     )
@@
     )
   )
-  (global_label "D13" (shape input) (at 208.28 90.17 0) (fields_autoplaced)
+  (global_label "D13" (shape input) (at 215.9 90.17 0) (fields_autoplaced)
     (effects (font (size 1.27 1.27)) (justify left))
-    (property "Intersheetrefs" "${INTERSHEET_REFS}" (at 214.9542 90.17 0)
+    (property "Intersheetrefs" "${INTERSHEET_REFS}" (at 222.5742 90.17 0)
       (effects (font (size 1.27 1.27)) (justify left) hide)
     )
@@
     )
   )
-  (global_label "D10" (shape input) (at 208.28 92.71 0) (fields_autoplaced)
+  (global_label "D10" (shape input) (at 215.9 92.71 0) (fields_autoplaced)
     (effects (font (size 1.27 1.27)) (justify left))
-    (property "Intersheetrefs" "${INTERSHEET_REFS}" (at 214.9542 92.71 0)
+    (property "Intersheetrefs" "${INTERSHEET_REFS}" (at 222.5742 92.71 0)
       (effects (font (size 1.27 1.27)) (justify left) hide)
     )
@@
     )
   )
-  (global_label "D12" (shape input) (at 208.28 87.63 0) (fields_autoplaced)
+  (global_label "D12" (shape input) (at 215.9 87.63 0) (fields_autoplaced)
     (effects (font (size 1.27 1.27)) (justify left))
-    (property "Intersheetrefs" "${INTERSHEET_REFS}" (at 214.9542 87.63 0)
+    (property "Intersheetrefs" "${INTERSHEET_REFS}" (at 222.5742 87.63 0)
       (effects (font (size 1.27 1.27)) (justify left) hide)
     )
@@
     )
   )
+  (symbol (lib_id "Device:R") (at 194.31 92.71 270) (unit 1)
+    (in_bom yes) (on_board yes) (dnp no)
+    (property "Reference" "R7" (at 199.39 93.98 90)
+      (effects (font (size 1.27 1.27)))
+    )
+    (property "Value" "0" (at 190.5 91.44 90)
+      (effects (font (size 1.27 1.27)))
+    )
+    (property "Footprint" "Resistor_SMD:R_0402_1005Metric" (at 194.31 90.932 90)
+      (effects (font (size 1.27 1.27)) hide)
+    )
+    (property "Datasheet" "~" (at 194.31 92.71 0)
+      (effects (font (size 1.27 1.27)) hide)
+    )
+    (pin "1")
+    (pin "2")
+    (instances
+      (project "central_hub"
+        (path "/0d9ec66e-0fbf-4d12-9b83-adf78971a00b/a9a7affa-d8a7-4dcd-8fe3-0de6a2b29bd6"
+          (reference "R7") (unit 1)
+        )
+        (path "/0d9ec66e-0fbf-4d12-9b83-adf78971a00b/4fb60496-ee10-4e45-a75e-a49c2c8afc68"
+          (reference "R37") (unit 1)
+        )
+      )
+      (project "motor_board_pcb"
+        (path "/4ad82a24-c992-45c9-b523-12e12bcd6ced"
+          (reference "R?") (unit 1)
+        )
+        (path "/4ad82a24-c992-45c9-b523-12e12bcd6ced/63c66207-e5d4-4f6f-af8f-451675dc3930"
+          (reference "R16") (unit 1)
+        )
+      )
+    )
+  )
   (symbol (lib_id "Device:C") (at 80.01 69.85 90) (unit 1)
     (in_bom yes) (on_board yes) (dnp no)
@@
         (path "/0d9ec66e-0fbf-4d12-9b83-adf78971a00b/4fb60496-ee10-4e45-a75e-a49c2c8afc68"
           (reference "C1") (unit 1)
+        )
+      )
+    )
+  )
+  (symbol (lib_id "Device:R") (at 194.31 85.09 270) (unit 1)
+    (in_bom yes) (on_board yes) (dnp no)
+    (property "Reference" "R7" (at 199.39 86.36 90)
+      (effects (font (size 1.27 1.27)))
+    )
+    (property "Value" "0" (at 190.5 83.82 90)
+      (effects (font (size 1.27 1.27)))
+    )
+    (property "Footprint" "Resistor_SMD:R_0402_1005Metric" (at 194.31 83.312 90)
+      (effects (font (size 1.27 1.27)) hide)
+    )
+    (property "Datasheet" "~" (at 194.31 85.09 0)
+      (effects (font (size 1.27 1.27)) hide)
+    )
+    (pin "1")
+    (pin "2")
+    (instances
+      (project "central_hub"
+        (path "/0d9ec66e-0fbf-4d12-9b83-adf78971a00b/a9a7affa-d8a7-4dcd-8fe3-0de6a2b29bd6"
+          (reference "R7") (unit 1)
+        )
+        (path "/0d9ec66e-0fbf-4d12-9b83-adf78971a00b/4fb60496-ee10-4e45-a75e-a49c2c8afc68"
+          (reference "R35") (unit 1)
+        )
+      )
+      (project "motor_board_pcb"
+        (path "/4ad82a24-c992-45c9-b523-12e12bcd6ced"
+          (reference "R?") (unit 1)
+        )
+        (path "/4ad82a24-c992-45c9-b523-12e12bcd6ced/63c66207-e5d4-4f6f-af8f-451675dc3930"
+          (reference "R16") (unit 1)
         )
       )
@@
         )
       )
+    )
+  )
+  (symbol (lib_id "Device:R") (at 194.31 90.17 270) (unit 1)
+    (in_bom yes) (on_board yes) (dnp no)
+    (property "Reference" "R7" (at 199.39 91.44 90)
+      (effects (font (size 1.27 1.27)))
+    )
+    (property "Value" "0" (at 190.5 88.9 90)
+      (effects (font (size 1.27 1.27)))
+    )
+    (property "Footprint" "Resistor_SMD:R_0402_1005Metric" (at 194.31 88.392 90)
+      (effects (font (size 1.27 1.27)) hide)
+    )
+    (property "Datasheet" "~" (at 194.31 90.17 0)
+      (effects (font (size 1.27 1.27)) hide)
+    )
+    (pin "1")
+    (pin "2")
+    (instances
+      (project "central_hub"
+        (path "/0d9ec66e-0fbf-4d12-9b83-adf78971a00b/a9a7affa-d8a7-4dcd-8fe3-0de6a2b29bd6"
+          (reference "R7") (unit 1)
+        )
+        (path "/0d9ec66e-0fbf-4d12-9b83-adf78971a00b/4fb60496-ee10-4e45-a75e-a49c2c8afc68"
+          (reference "R36") (unit 1)
+        )
+      )
+      (project "motor_board_pcb"
+        (path "/4ad82a24-c992-45c9-b523-12e12bcd6ced"
+          (reference "R?") (unit 1)
+        )
+        (path "/4ad82a24-c992-45c9-b523-12e12bcd6ced/63c66207-e5d4-4f6f-af8f-451675dc3930"
+          (reference "R16") (unit 1)
+        )
+      )

Commit message: Kim changes
Parts:
- removed D7: LED, Diode_SMD:D_0603_1608Metric, symbol Device:LED
- removed R15: 330, Resistor_SMD:R_0603_1608Metric, symbol Device:R
- C1, C2: value 15pF -> 22p
- Y1: value 16MHz -> 8M
Other:
- note removed: "SCK LED"
Changed lines of the file:
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@@
-    (stroke (width 0) (type default))
-  )
-  (wire (pts (xy 165.1 176.53) (xy 165.1 177.8))
     (stroke (width 0) (type default))
   )
@@
     (stroke (width 0) (type default))
   )
-  (wire (pts (xy 165.1 185.42) (xy 165.1 186.69))
-    (stroke (width 0) (type default))
-  )
   (wire (pts (xy 233.68 102.87) (xy 233.68 97.79))
     (stroke (width 0) (type default))
@@
     (stroke (width 0) (type default))
   )
-  (wire (pts (xy 165.1 168.91) (xy 165.1 166.37))
-    (stroke (width 0) (type default))
-  )
   (wire (pts (xy 73.66 96.52) (xy 73.66 97.79))
     (stroke (width 0) (type default))
@@
     (stroke (width 0) (type default))
   )
-  (wire (pts (xy 151.13 166.37) (xy 165.1 166.37))
-    (stroke (width 0) (type default))
-  )
   (wire (pts (xy 93.98 92.71) (xy 119.38 92.71))
     (stroke (width 0) (type default))
@@
   (wire (pts (xy 72.39 69.85) (xy 76.2 69.85))
     (stroke (width 0) (type default))
-  )
-  (text "YELLOW" (at 168.91 179.07 0)
-    (effects (font (size 1.27 1.27) (color 194 194 0 1)) (justify left bottom))
   )
   (text "TX\nLED" (at 102.87 161.29 0)
@@
     (effects (font (size 1.27 1.27) (color 194 194 0 1)) (justify left bottom))
   )
-  (text "SCK\nLED" (at 161.29 161.29 0)
-    (effects (font (size 2.54 2.54) (thickness 0.254) bold) (justify left bottom))
-  )
   (text "USB LDO OUTPUT\n" (at 87.63 80.01 0)
     (effects (font (size 1.27 1.27) (thickness 0.254) bold) (justify left bottom))
@@
   )
   (label "P303_GPT7_B" (at 191.77 120.65 0) (fields_autoplaced)
-    (effects (font (size 1.27 1.27)) (justify left bottom))
-  )
-  (label "P111_GPT3_A" (at 151.13 166.37 0) (fields_autoplaced)
     (effects (font (size 1.27 1.27)) (justify left bottom))
   )
@@
       (effects (font (size 1.27 1.27)))
     )
-    (property "Value" "15pF" (at 80.01 29.21 90)
+    (property "Value" "22p" (at 80.01 29.21 90)
       (effects (font (size 1.27 1.27)))
     )
@@
         (path "/0d9ec66e-0fbf-4d12-9b83-adf78971a00b/4fb60496-ee10-4e45-a75e-a49c2c8afc68"
           (reference "TP5") (unit 1)
-        )
-      )
-    )
-  )
-  (symbol (lib_id "Device:LED") (at 165.1 172.72 90) (unit 1)
-    (in_bom yes) (on_board yes) (dnp no) (fields_autoplaced)
-    (property "Reference" "D7" (at 168.91 173.0375 90)
-      (effects (font (size 1.27 1.27)) (justify right))
-    )
-    (property "Value" "LED" (at 168.91 175.5775 90)
-      (effects (font (size 1.27 1.27)) (justify right))
-    )
-    (property "Footprint" "Diode_SMD:D_0603_1608Metric" (at 165.1 172.72 0)
-      (effects (font (size 1.27 1.27)) hide)
-    )
-    (property "Datasheet" "~" (at 165.1 172.72 0)
-      (effects (font (size 1.27 1.27)) hide)
-    )
-    (pin "1")
-    (pin "2")
-    (instances
-      (project "central_hub"
-        (path "/0d9ec66e-0fbf-4d12-9b83-adf78971a00b"
-          (reference "D7") (unit 1)
-        )
-        (path "/0d9ec66e-0fbf-4d12-9b83-adf78971a00b/4fb60496-ee10-4e45-a75e-a49c2c8afc68"
-          (reference "D4") (unit 1)
         )
       )
@@
     )
   )
-  (symbol (lib_id "power:GND") (at 165.1 186.69 0) (unit 1)
-    (in_bom yes) (on_board yes) (dnp no)
-    (property "Reference" "#PWR040" (at 165.1 193.04 0)
-      (effects (font (size 1.27 1.27)) hide)
-    )
-    (property "Value" "GND" (at 165.1 191.77 0)
-      (effects (font (size 1.27 1.27)))
-    )
-    (property "Footprint" "" (at 165.1 186.69 0)
-      (effects (font (size 1.27 1.27)) hide)
-    )
-    (property "Datasheet" "" (at 165.1 186.69 0)
-      (effects (font (size 1.27 1.27)) hide)
-    )
-    (pin "1")
-    (instances
-      (project "central_hub"
-        (path "/0d9ec66e-0fbf-4d12-9b83-adf78971a00b"
-          (reference "#PWR040") (unit 1)
-        )
-        (path "/0d9ec66e-0fbf-4d12-9b83-adf78971a00b/4fb60496-ee10-4e45-a75e-a49c2c8afc68"
-          (reference "#PWR027") (unit 1)
-        )
-      )
-    )
-  )
   (symbol (lib_id "power:GND") (at 72.39 59.69 270) (unit 1)
     (in_bom yes) (on_board yes) (dnp no) (fields_autoplaced)
@@
       (effects (font (size 1.27 1.27)) (justify right))
     )
-    (property "Value" "16MHz" (at 96.52 44.45 90)
+    (property "Value" "8M" (at 96.52 44.45 90)
       (effects (font (size 1.27 1.27)) (justify right))
     )
@@
       (effects (font (size 1.27 1.27)))
     )
-    (property "Value" "15pF" (at 80.01 46.99 90)
+    (property "Value" "22p" (at 80.01 46.99 90)
       (effects (font (size 1.27 1.27)))
     )
@@
         )
       )
-    )
-  )
-  (symbol (lib_id "Device:R") (at 165.1 181.61 0) (unit 1)
-    (in_bom yes) (on_board yes) (dnp no) (fields_autoplaced)
-    (property "Reference" "R15" (at 167.64 180.34 0)
-      (effects (font (size 1.27 1.27)) (justify left))
-    )
-    (property "Value" "330" (at 167.64 182.88 0)
-      (effects (font (size 1.27 1.27)) (justify left))
-    )
-    (property "Footprint" "Resistor_SMD:R_0603_1608Metric" (at 163.322 181.61 90)
-      (effects (font (size 1.27 1.27)) hide)
-    )
-    (property "Datasheet" "~" (at 165.1 181.61 0)
-      (effects (font (size 1.27 1.27)) hide)
-    )
-    (pin "1")
-    (pin "2")
-    (instances
-      (project "central_hub"
-        (path "/0d9ec66e-0fbf-4d12-9b83-adf78971a00b"
-          (reference "R15") (unit 1)
-        )
-        (path "/0d9ec66e-0fbf-4d12-9b83-adf78971a00b/4fb60496-ee10-4e45-a75e-a49c2c8afc68"
-          (reference "R11") (unit 1)
-        )
-      )

Commit message: - added footprint labels to schematic
Parts:
- C1, C2, C3, C4, C5, R16: fp (none) -> 0603
- C10, C6, C7, C8, C9, D3, D5, D6, L1, L2, R1, R10, R11, R12, R13, R14, R2, R3, R5, R6, R7, R8: FP (none) -> 0603
- R7: FP (none) -> 0402
