File: Hub_Board_PCB/central_hub/central_hub.kicad_pcb (KiCad board)
At the start: 2 copper layers, 108 x 61.7 mm, 117 parts, among them J1 CAN_OUT, J2 Conn_01x02, J3 Screw_Terminal_01x08, J4 Screw_Terminal_01x08, J5 CSP-USC16-TR, J6 Screw_Terminal_01x04, J7 Conn_01x03, J8 Conn_01x02, J9 Screw_Terminal_01x04, Q1 BSS138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

Commit message: Kim changes
Parts:
- removed D4: LED, Diode_SMD:D_0603_1608Metric
- added C32: 0.1u, Capacitor_SMD:C_0402_1005Metric, F.Cu at (102.1, 79.9)
- C11, C13: value 15p -> 22p
- C2, C3: value 15pF -> 22p
- R11: value 330 -> 0; footprint Resistor_SMD:R_0603_1608Metric -> Resistor_SMD:R_0402_1005Metric
- Y1: value 16MHz -> 8M
- Y2: value 20M -> 8M
- moved R11 23.3 mm to (101.7, 78.5), turned to 90 degrees
- moved TP5 0.86 mm to (100.5, 62.5)
Connections:
- R11 pad 1: Net-(D4-K) -> Net-(U3-SCK)
- R11 pad 2: GND -> D13
- U3 pad 14: D13 -> Net-(U3-SCK)
Routing:
- net D13: track 94.1 -> 62.4 mm, vias 6 -> 4
- net Net-(U3-SCK): track 0.00 -> 2.25 mm
- net Net-(D4-K): track 1.69 -> 0.00 mm
- net GND: track 52.2 -> 51.8 mm, vias 80 -> 373
