File: Motor_Board_PCB/motor_board_pcb/Connectors_Sheet.kicad_sch (KiCad schematic)
At the start: 10 parts, among them J11 CSP-USC16-TR, J6 Screw_Terminal_01x04, J7 Conn_01x03, J8 Conn_01x02

Commit message: Motor Board Initial Layout
Parts:
- removed J?: Screw_Terminal_01x14, Connector_PinHeader_2.54mm:PinHeader_1x14_P2.54mm_Vertical, symbol Connector:Screw_Terminal_01x14
- added J4: Screw_Terminal_01x06, Connector_PinHeader_2.54mm:PinHeader_1x06_P2.54mm_Vertical, symbol Connector:Screw_Terminal_01x06
- added TP? (x8): TestPoint, TestPoint:TestPoint_Pad_D1.0mm, symbol Connector:TestPoint
Connections:
- net +5V: now also J4.1 (Pin_1)
- net D0: now also TP?.1
- net D1: now also TP?.1
- net D10: now also TP?.1
- net D11: now also TP?.1
- net D12: now also TP?.1
- net D13: now also TP?.1
- net D2: now also J4.5 (Pin_5)
- net D3: now also J4.4 (Pin_4)
- net D4: now also J4.3 (Pin_3)
- net D5: now also J4.2 (Pin_2)
- net D6: now also TP?.1
- net D7: now also TP?.1
- net GND: now also J4.6 (Pin_6)

Commit message: All usb changes on both boards
Parts:
- removed TP? (x2): TestPoint, TestPoint:TestPoint_Pad_D1.0mm, symbol Connector:TestPoint
Changed lines of the file:
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@@
-    )
-  )
-  (symbol (lib_id "Connector:TestPoint") (at 93.98 101.6 270) (mirror x) (unit 1)
-    (in_bom yes) (on_board yes) (dnp no)
-    (property "Reference" "TP?" (at 101.6 101.6 90)
-      (effects (font (size 1.27 1.27)))
-    )
-    (property "Value" "TestPoint" (at 97.282 99.06 90)
-      (effects (font (size 1.27 1.27)) hide)
-    )
-    (property "Footprint" "TestPoint:TestPoint_Pad_D1.0mm" (at 93.98 96.52 0)
-      (effects (font (size 1.27 1.27)) hide)
-    )
-    (property "Datasheet" "~" (at 93.98 96.52 0)
-      (effects (font (size 1.27 1.27)) hide)
-    )
-    (pin "1")
-    (instances
-      (project "central_hub"
-        (path "/0d9ec66e-0fbf-4d12-9b83-adf78971a00b"
-          (reference "TP?") (unit 1)
-        )
-        (path "/0d9ec66e-0fbf-4d12-9b83-adf78971a00b/4fb60496-ee10-4e45-a75e-a49c2c8afc68"
-          (reference "TP?") (unit 1)
-        )
-        (path "/0d9ec66e-0fbf-4d12-9b83-adf78971a00b/8e53aed1-21e6-440d-aae4-1b5509ec346a"
-          (reference "TP?") (unit 1)
-        )
-      )
-      (project "motor_board_pcb"
-        (path "/4ad82a24-c992-45c9-b523-12e12bcd6ced/996060af-581e-425f-9e10-26ee39d5a960"
-          (reference "TP7") (unit 1)
-        )
-      )
     )
   )
@@
         )
       )
-    )
-  )
-  (symbol (lib_id "Connector:TestPoint") (at 93.98 104.14 270) (mirror x) (unit 1)
-    (in_bom yes) (on_board yes) (dnp no)
-    (property "Reference" "TP?" (at 101.6 104.14 90)
-      (effects (font (size 1.27 1.27)))
-    )
-    (property "Value" "TestPoint" (at 97.282 101.6 90)
-      (effects (font (size 1.27 1.27)) hide)
-    )
-    (property "Footprint" "TestPoint:TestPoint_Pad_D1.0mm" (at 93.98 99.06 0)
-      (effects (font (size 1.27 1.27)) hide)
-    )
-    (property "Datasheet" "~" (at 93.98 99.06 0)
-      (effects (font (size 1.27 1.27)) hide)
-    )
-    (pin "1")
-    (instances
-      (project "central_hub"
-        (path "/0d9ec66e-0fbf-4d12-9b83-adf78971a00b"
-          (reference "TP?") (unit 1)
-        )
-        (path "/0d9ec66e-0fbf-4d12-9b83-adf78971a00b/4fb60496-ee10-4e45-a75e-a49c2c8afc68"
-          (reference "TP?") (unit 1)
-        )
-        (path "/0d9ec66e-0fbf-4d12-9b83-adf78971a00b/8e53aed1-21e6-440d-aae4-1b5509ec346a"
-          (reference "TP?") (unit 1)
-        )
-      )
-      (project "motor_board_pcb"
-        (path "/4ad82a24-c992-45c9-b523-12e12bcd6ced/996060af-581e-425f-9e10-26ee39d5a960"
-          (reference "TP8") (unit 1)
-        )
-      )

Commit message: - added footprint labels to schematic symbols
Parts:
- C?, R?: FP (none) -> 0603
Changed lines of the file:
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@@
       (effects (font (size 1.27 1.27)) hide)
+    )
+    (property "FP" "0603" (at 90.17 130.81 0)
+      (effects (font (size 1.27 1.27)))
     )
     (pin "1")
@@
   )
   (symbol (lib_id "Device:R") (at 96.52 127 0) (unit 1)
-    (in_bom yes) (on_board yes) (dnp no) (fields_autoplaced)
+    (in_bom yes) (on_board yes) (dnp no)
     (property "Reference" "R?" (at 99.06 125.73 0)
       (effects (font (size 1.27 1.27)) (justify left))
@@
       (effects (font (size 1.27 1.27)) hide)
     )
+    (property "FP" "0603" (at 101.6 130.81 0)
+      (effects (font (size 1.27 1.27)))
+    )
     (pin "1")
