File: Motor_Board_PCB/motor_board_pcb/Motor_Driver_Sheet.kicad_sch (KiCad schematic)
At the start: 0 parts

Commit message: Added power and motor driver chip schematics
Parts:
- added C26, C27, C32: 4u7, symbol Device:C
- added C28, C30, C31, C33: 100n, symbol Device:C
- added C29: 22n, symbol Device:C
- added J7: Screw_Terminal_01x04, symbol Connector:Screw_Terminal_01x04
- added R17, R18, R19, R20, R21, R24: 10K, symbol Device:R
- added R22, R23: 2k, symbol Device:R
- added R25: 100K, symbol Device:R
- added R26, R27: 0R11, symbol Device:R
- added RV1: 10K, symbol Device:R_Potentiometer
- added U5: TMC2209-LA, QFN28_5X5_TRI, symbol TMC2209-LA:TMC2209-LA
Connections:
- new net: R17.2, U5.2 (!ENN)
- new net: R24.2, U5.14 (PDN_UART)
- new net: R19.2, U5.10 (MS2_AD1)
- new net: R22.1, U5.19 (DIR)
- new net: R20.1, RV1.1
- new net: RV1.2, U5.17 (VREF)
- new net: R23.1, U5.16 (STEP)
- new net: R27.2, U5.23 (BRA)
- new net: C31.1, U5.6 (VCP)
- new net: R21.2, U5.7 (SPREAD)
- new net: R25.2, U5.20 (STDBY)
- new net: R18.2, U5.9 (MS1_AD0)
- new net: R26.2, U5.27 (BRB)
- new net: C29.2, U5.4 (CPO)
- new net: C29.1, U5.5 (CPI)
- new net +12V: C26.2, C27.2, C28.2, C30.2, C31.2, U5.22 (VS), U5.28 (VS)
- new net +5V: C33.1, U5.15 (VCC_IO)
- new net 5VOUT: C32.2, R20.2, U5.8 (5VOUT)
- new net D_DIR: R22.2
- new net D_STEP: R23.2
- new net GND: C26.1, C27.1, C28.1, C30.1, C32.1, C33.2, R17.1, R18.1, R19.1, R21.1, R24.1, R25.1, R26.1, R27.1, RV1.3, U5.13 (CLK), U5.18 (GND), U5.29 (GND), U5.3 (GND)
- new net OUTA1: J7.3 (Pin_3), U5.24 (OUTA1)
- new net OUTA2: J7.4 (Pin_4), U5.21 (OUTA2)
- new net OUTB1: J7.2 (Pin_2), U5.26 (OUTB1)
- new net OUTB2: J7.1 (Pin_1), U5.1 (OUTB2)
- no-connect marks 0 -> 2

Commit message: Added footprints for almost all components
Parts:
- C15: renamed from C26; footprint (none) -> Capacitor_SMD:C_0603_1608Metric
- C16: renamed from C27; footprint (none) -> Capacitor_SMD:C_0603_1608Metric
- C17: renamed from C28; footprint (none) -> Capacitor_SMD:C_0603_1608Metric
- C18: renamed from C29; footprint (none) -> Capacitor_SMD:C_0603_1608Metric
- C19: renamed from C30; footprint (none) -> Capacitor_SMD:C_0603_1608Metric
- C20: renamed from C31; footprint (none) -> Capacitor_SMD:C_0603_1608Metric
- C21: renamed from C32; footprint (none) -> Capacitor_SMD:C_0603_1608Metric
- C22: renamed from C33; footprint (none) -> Capacitor_SMD:C_0603_1608Metric
- J2: renamed from J7; footprint (none) -> Connector_PinHeader_1.00mm:PinHeader_1x04_P1.00mm_Vertical
- R19: renamed from R17; footprint (none) -> Resistor_SMD:R_0603_1608Metric
- R20: renamed from R18; footprint (none) -> Resistor_SMD:R_0603_1608Metric
- R21: renamed from R19; footprint (none) -> Resistor_SMD:R_0603_1608Metric
- R22: renamed from R20; footprint (none) -> Resistor_SMD:R_0603_1608Metric
- R23: renamed from R21; footprint (none) -> Resistor_SMD:R_0603_1608Metric
- R24: renamed from R22; footprint (none) -> Resistor_SMD:R_0603_1608Metric
- R25: renamed from R23; footprint (none) -> Resistor_SMD:R_0603_1608Metric
- R26: renamed from R24; footprint (none) -> Resistor_SMD:R_0603_1608Metric
- R27: renamed from R25; footprint (none) -> Resistor_SMD:R_0603_1608Metric
- R28: renamed from R26; footprint (none) -> Resistor_SMD:R_0603_1608Metric
- R29: renamed from R27; footprint (none) -> Resistor_SMD:R_0603_1608Metric
- U4: renamed from U5; footprint QFN28_5X5_TRI -> (none)

Commit message: Added all other footprints... populated all components with NO errors or warnings :)
Parts:
- RV1: footprint (none) -> ~ALL:TRIM_TC33X-2-103E
- U4: footprint (none) -> ~ALL:QFN50P500X500X90-29N
Changed lines of the file:
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@@
       (effects (font (size 1.27 1.27)) (justify right))
     )
-    (property "Footprint" "" (at 50.8 101.6 0)
+    (property "Footprint" "~ALL:TRIM_TC33X-2-103E" (at 50.8 101.6 0)
       (effects (font (size 1.27 1.27)) hide)
     )
@@
       (effects (font (size 1.524 1.524)) (justify left))
     )
-    (property "Footprint" "" (at 116.84 81.28 0)
+    (property "Footprint" "~ALL:QFN50P500X500X90-29N" (at 116.84 81.28 0)
       (effects (font (size 1.27 1.27) italic) hide)
     )

Commit message: Fixed header sizes
Parts:
- J2: footprint Connector_PinHeader_1.00mm:PinHeader_1x04_P1.00mm_Vertical -> Connector_PinHeader_2.54mm:PinHeader_1x04_P2.54mm_Vertical
Changed lines of the file:
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@@
       (effects (font (size 1.27 1.27)) (justify left))
     )
-    (property "Footprint" "Connector_PinHeader_1.00mm:PinHeader_1x04_P1.00mm_Vertical" (at 158.75 63.5 0)
+    (property "Footprint" "Connector_PinHeader_2.54mm:PinHeader_1x04_P2.54mm_Vertical" (at 158.75 63.5 0)
       (effects (font (size 1.27 1.27)) hide)
     )

Commit message: Initial PCB placement for Motor Board
Parts:
- C17, C18, C19, C20, C22: footprint Capacitor_SMD:C_0603_1608Metric -> Capacitor_SMD:C_0402_1005Metric
Connections:
- net D_DIR renamed D7
- net D_STEP renamed D6
Changed lines of the file:
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@@
     (stroke (width 0) (type default))
   )
-  (wire (pts (xy 59.69 71.12) (xy 66.04 71.12))
+  (wire (pts (xy 60.96 71.12) (xy 66.04 71.12))
     (stroke (width 0) (type default))
   )
@@
     (effects (font (size 1.27 1.27)) (justify right bottom))
   )
-  (global_label "D_DIR" (shape input) (at 59.69 71.12 180) (fields_autoplaced)
+  (global_label "D7" (shape input) (at 60.96 71.12 180) (fields_autoplaced)
     (effects (font (size 1.27 1.27)) (justify right))
-    (property "Intersheetrefs" "${INTERSHEET_REFS}" (at 51.3224 71.12 0)
+    (property "Intersheetrefs" "${INTERSHEET_REFS}" (at 55.4953 71.12 0)
       (effects (font (size 1.27 1.27)) (justify right) hide)
     )
   )
-  (global_label "D_STEP" (shape input) (at 60.96 73.66 180) (fields_autoplaced)
+  (global_label "D6" (shape input) (at 60.96 73.66 180) (fields_autoplaced)
     (effects (font (size 1.27 1.27)) (justify right))
-    (property "Intersheetrefs" "${INTERSHEET_REFS}" (at 51.1411 73.66 0)
+    (property "Intersheetrefs" "${INTERSHEET_REFS}" (at 55.4953 73.66 0)
       (effects (font (size 1.27 1.27)) (justify right) hide)
     )
@@
       (effects (font (size 1.27 1.27)) (justify right))
     )
-    (property "Footprint" "Capacitor_SMD:C_0603_1608Metric" (at 75.2348 35.56 0)
+    (property "Footprint" "Capacitor_SMD:C_0402_1005Metric" (at 75.2348 35.56 0)
       (effects (font (size 1.27 1.27)) hide)
     )
@@
       (effects (font (size 1.27 1.27)))
     )
-    (property "Footprint" "Capacitor_SMD:C_0603_1608Metric" (at 110.49 35.2552 0)
+    (property "Footprint" "Capacitor_SMD:C_0402_1005Metric" (at 110.49 35.2552 0)
       (effects (font (size 1.27 1.27)) hide)
     )
@@
       (effects (font (size 1.27 1.27)) (justify left))
     )
-    (property "Footprint" "Capacitor_SMD:C_0603_1608Metric" (at 154.6352 90.17 0)
+    (property "Footprint" "Capacitor_SMD:C_0402_1005Metric" (at 154.6352 90.17 0)
       (effects (font (size 1.27 1.27)) hide)
     )
@@
       (effects (font (size 1.27 1.27)) (justify right))
     )
-    (property "Footprint" "Capacitor_SMD:C_0603_1608Metric" (at 87.9348 35.56 0)
+    (property "Footprint" "Capacitor_SMD:C_0402_1005Metric" (at 87.9348 35.56 0)
       (effects (font (size 1.27 1.27)) hide)
     )
@@
       (effects (font (size 1.27 1.27)) (justify right))
     )
-    (property "Footprint" "Capacitor_SMD:C_0603_1608Metric" (at 82.8548 53.34 0)
-      (effects (font (size 1.27 1.27)) hide)
-    )
+    (property "Footprint" "Capacitor_SMD:C_0402_1005Metric" (at 82.8548 53.34 0)
+      (effects (font (size 1.27 1.27)) hide)
+    )

Commit message: Schematic changes before sending to kim
Parts:
- added R31, R32, R33: 10K, Resistor_SMD:R_0603_1608Metric, symbol Device:R
Connections:
- net +5V: now also R31.2, R32.2, R33.2
- net at R23.2, U4.7 (SPREAD): now also R33.1
- net at R20.2, U4.9 (MS1_AD0): now also R31.1, R32.1
Changed lines of the file:
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@@
 (kicad_sch (version 20230121) (generator eeschema)
   (paper "A4")
+  (junction (at 69.85 91.44) (diameter 0) (color 0 0 0 0)
+  )
   (junction (at 104.14 34.29) (diameter 0) (color 0 0 0 0)
   )
@@
   (junction (at 153.67 78.74) (diameter 0) (color 0 0 0 0)
   )
+  (junction (at 38.1 78.74) (diameter 0) (color 0 0 0 0)
+  )
   (junction (at 106.68 34.29) (diameter 0) (color 0 0 0 0)
   )
   (junction (at 76.2 34.29) (diameter 0) (color 0 0 0 0)
+  )
+  (junction (at 30.48 78.74) (diameter 0) (color 0 0 0 0)
   )
   (junction (at 106.68 107.95) (diameter 0) (color 0 0 0 0)
@@
     (stroke (width 0) (type default))
   )
+  (wire (pts (xy 45.72 62.23) (xy 45.72 82.55))
+    (stroke (width 0) (type default))
+  )
   (wire (pts (xy 83.82 99.06) (xy 83.82 102.87))
     (stroke (width 0) (type default))
@@
     (stroke (width 0) (type default))
   )
-  (wire (pts (xy 29.21 78.74) (xy 91.44 78.74))
+  (wire (pts (xy 29.21 78.74) (xy 30.48 78.74))
+    (stroke (width 0) (type default))
+  )
+  (wire (pts (xy 30.48 50.8) (xy 30.48 54.61))
     (stroke (width 0) (type default))
   )
@@
     (stroke (width 0) (type default))
   )
-  (wire (pts (xy 91.44 91.44) (xy 66.04 91.44))
+  (wire (pts (xy 91.44 91.44) (xy 69.85 91.44))
     (stroke (width 0) (type default))
   )
@@
     (stroke (width 0) (type default))
   )
+  (wire (pts (xy 69.85 82.55) (xy 69.85 91.44))
+    (stroke (width 0) (type default))
+  )
   (wire (pts (xy 60.96 71.12) (xy 66.04 71.12))
     (stroke (width 0) (type default))
   )
+  (wire (pts (xy 45.72 82.55) (xy 69.85 82.55))
+    (stroke (width 0) (type default))
+  )
   (wire (pts (xy 118.11 107.95) (xy 118.11 106.68))
     (stroke (width 0) (type default))
   )
+  (wire (pts (xy 38.1 62.23) (xy 38.1 78.74))
+    (stroke (width 0) (type default))
+  )
   (wire (pts (xy 115.57 107.95) (xy 118.11 107.95))
     (stroke (width 0) (type default))
@@
     (stroke (width 0) (type default))
   )
+  (wire (pts (xy 38.1 50.8) (xy 38.1 54.61))
+    (stroke (width 0) (type default))
+  )
   (wire (pts (xy 88.9 34.29) (xy 104.14 34.29))
     (stroke (width 0) (type default))
@@
     (stroke (width 0) (type default))
   )
+  (wire (pts (xy 69.85 91.44) (xy 66.04 91.44))
+    (stroke (width 0) (type default))
+  )
   (wire (pts (xy 153.67 78.74) (xy 153.67 82.55))
     (stroke (width 0) (type default))
@@
     (stroke (width 0) (type default))
   )
+  (wire (pts (xy 30.48 62.23) (xy 30.48 78.74))
+    (stroke (width 0) (type default))
+  )
+  (wire (pts (xy 30.48 78.74) (xy 38.1 78.74))
+    (stroke (width 0) (type default))
+  )
   (wire (pts (xy 83.82 63.5) (xy 91.44 63.5))
     (stroke (width 0) (type default))
@@
     (stroke (width 0) (type default))
   )
+  (wire (pts (xy 38.1 78.74) (xy 91.44 78.74))
+    (stroke (width 0) (type default))
+  )
   (wire (pts (xy 88.9 34.29) (xy 88.9 35.56))
     (stroke (width 0) (type default))
@@
   )
   (wire (pts (xy 66.04 91.44) (xy 66.04 102.87))
+    (stroke (width 0) (type default))
+  )
+  (wire (pts (xy 45.72 50.8) (xy 45.72 54.61))
     (stroke (width 0) (type default))
   )
@@
     )
   )
+  (symbol (lib_id "Device:R") (at 38.1 58.42 180) (unit 1)
+    (in_bom yes) (on_board yes) (dnp yes) (fields_autoplaced)
+    (property "Reference" "R31" (at 40.64 57.15 0)
+      (effects (font (size 1.27 1.27)) (justify right))
+    )
+    (property "Value" "10K" (at 40.64 59.69 0)
+      (effects (font (size 1.27 1.27)) (justify right))
+    )
+    (property "Footprint" "Resistor_SMD:R_0603_1608Metric" (at 39.878 58.42 90)
+      (effects (font (size 1.27 1.27)) hide)
+    )
+    (property "Datasheet" "~" (at 38.1 58.42 0)
+      (effects (font (size 1.27 1.27)) hide)
+    )
+    (pin "1")
+    (pin "2")
+    (instances
+      (project "motor_board_pcb"
+        (path "/4ad82a24-c992-45c9-b523-12e12bcd6ced/b57f9924-5c2c-40da-8939-31af087f9aa3"
+          (reference "R31") (unit 1)
+        )
+      )
+      (project "LocalDesign"
+        (path "/a439ee58-92e3-49e0-a19d-7c5a25d23ba1"
+          (reference "R?") (unit 1)
+        )
+      )
+    )
+  )
   (symbol (lib_id "power:+5V") (at 153.67 78.74 0) (unit 1)
     (in_bom yes) (on_board yes) (dnp no) (fields_autoplaced)
@@
         (path "/4ad82a24-c992-45c9-b523-12e12bcd6ced/b57f9924-5c2c-40da-8939-31af087f9aa3"
           (reference "#PWR053") (unit 1)
+        )
+      )
+      (project "LocalDesign"
+        (path "/a439ee58-92e3-49e0-a19d-7c5a25d23ba1"
+          (reference "#PWR?") (unit 1)
+        )
+      )
+    )
+  )
+  (symbol (lib_id "power:+5V") (at 38.1 50.8 0) (unit 1)
+    (in_bom yes) (on_board yes) (dnp no) (fields_autoplaced)
+    (property "Reference" "#PWR062" (at 38.1 54.61 0)
+      (effects (font (size 1.27 1.27)) hide)
+    )
+    (property "Value" "+5V" (at 38.1 45.72 0)
+      (effects (font (size 1.27 1.27)))
+    )
+    (property "Footprint" "" (at 38.1 50.8 0)
+      (effects (font (size 1.27 1.27)) hide)
+    )
+    (property "Datasheet" "" (at 38.1 50.8 0)
+      (effects (font (size 1.27 1.27)) hide)
+    )
+    (pin "1")
+    (instances
+      (project "motor_board_pcb"
+        (path "/4ad82a24-c992-45c9-b523-12e12bcd6ced/b57f9924-5c2c-40da-8939-31af087f9aa3"
+          (reference "#PWR062") (unit 1)
+        )
+      )
+      (project "LocalDesign"
+        (path "/a439ee58-92e3-49e0-a19d-7c5a25d23ba1"
+          (reference "#PWR?") (unit 1)
+        )
+      )
+    )
+  )
+  (symbol (lib_id "power:+5V") (at 45.72 50.8 0) (unit 1)
+    (in_bom yes) (on_board yes) (dnp no) (fields_autoplaced)
+    (property "Reference" "#PWR064" (at 45.72 54.61 0)
+      (effects (font (size 1.27 1.27)) hide)
+    )
+    (property "Value" "+5V" (at 45.72 45.72 0)
+      (effects (font (size 1.27 1.27)))
+    )
+    (property "Footprint" "" (at 45.72 50.8 0)
+      (effects (font (size 1.27 1.27)) hide)
+    )
+    (property "Datasheet" "" (at 45.72 50.8 0)
+      (effects (font (size 1.27 1.27)) hide)
+    )
+    (pin "1")
+    (instances
+      (project "motor_board_pcb"
+        (path "/4ad82a24-c992-45c9-b523-12e12bcd6ced/b57f9924-5c2c-40da-8939-31af087f9aa3"
+          (reference "#PWR064") (unit 1)
         )
       )
@@
     )
   )
+  (symbol (lib_id "power:+5V") (at 30.48 50.8 0) (unit 1)
+    (in_bom yes) (on_board yes) (dnp no) (fields_autoplaced)
+    (property "Reference" "#PWR058" (at 30.48 54.61 0)
+      (effects (font (size 1.27 1.27)) hide)
+    )
+    (property "Value" "+5V" (at 30.48 45.72 0)
+      (effects (font (size 1.27 1.27)))
+    )
+    (property "Footprint" "" (at 30.48 50.8 0)
+      (effects (font (size 1.27 1.27)) hide)
+    )
+    (property "Datasheet" "" (at 30.48 50.8 0)
+      (effects (font (size 1.27 1.27)) hide)
+    )
+    (pin "1")
+    (instances
+      (project "motor_board_pcb"
+        (path "/4ad82a24-c992-45c9-b523-12e12bcd6ced/b57f9924-5c2c-40da-8939-31af087f9aa3"
+          (reference "#PWR058") (unit 1)
+        )
+      )
+      (project "LocalDesign"
+        (path "/a439ee58-92e3-49e0-a19d-7c5a25d23ba1"
+          (reference "#PWR?") (unit 1)
+        )
+      )
+    )
+  )
   (symbol (lib_id "power:GND") (at 137.16 111.76 0) (unit 1)
     (in_bom yes) (on_board yes) (dnp no) (fields_autoplaced)
@@
         (path "/a439ee58-92e3-49e0-a19d-7c5a25d23ba1"
           (reference "#PWR?") (unit 1)
+        )
+      )
+    )
+  )
+  (symbol (lib_id "Device:R") (at 45.72 58.42 180) (unit 1)
+    (in_bom yes) (on_board yes) (dnp yes) (fields_autoplaced)
+    (property "Reference" "R33" (at 48.26 57.15 0)
+      (effects (font (size 1.27 1.27)) (justify right))
+    )
+    (property "Value" "10K" (at 48.26 59.69 0)
+      (effects (font (size 1.27 1.27)) (justify right))
+    )
+    (property "Footprint" "Resistor_SMD:R_0603_1608Metric" (at 47.498 58.42 90)
+      (effects (font (size 1.27 1.27)) hide)
+    )
+    (property "Datasheet" "~" (at 45.72 58.42 0)
+      (effects (font (size 1.27 1.27)) hide)
+    )
+    (pin "1")
+    (pin "2")
+    (instances
+      (project "motor_board_pcb"
+        (path "/4ad82a24-c992-45c9-b523-12e12bcd6ced/b57f9924-5c2c-40da-8939-31af087f9aa3"
+          (reference "R33") (unit 1)
+        )
+      )
+      (project "LocalDesign"
+        (path "/a439ee58-92e3-49e0-a19d-7c5a25d23ba1"
+          (reference "R?") (unit 1)
         )
       )
@@
         )
       )
+      (project "LocalDesign"
+        (path "/a439ee58-92e3-49e0-a19d-7c5a25d23ba1"
+          (reference "R?") (unit 1)
+        )
+      )
+    )
+  )
+  (symbol (lib_id "Device:R") (at 30.48 58.42 180) (unit 1)
+    (in_bom yes) (on_board yes) (dnp yes) (fields_autoplaced)
+    (property "Reference" "R32" (at 33.02 57.15 0)
+      (effects (font (size 1.27 1.27)) (justify right))
+    )
+    (property "Value" "10K" (at 33.02 59.69 0)
+      (effects (font (size 1.27 1.27)) (justify right))
+    )
+    (property "Footprint" "Resistor_SMD:R_0603_1608Metric" (at 32.258 58.42 90)
+      (effects (font (size 1.27 1.27)) hide)
+    )
+    (property "Datasheet" "~" (at 30.48 58.42 0)
+      (effects (font (size 1.27 1.27)) hide)
+    )
+    (pin "1")
+    (pin "2")
+    (instances
+      (project "motor_board_pcb"
+        (path "/4ad82a24-c992-45c9-b523-12e12bcd6ced/b57f9924-5c2c-40da-8939-31af087f9aa3"
+          (reference "R32") (unit 1)
+        )
+      )

Commit message: Motor Board Initial Layout
Connections:
- net at R21.2, U4.10 (MS2_AD1): now also R31.1
- net at R20.2, R32.1, U4.9 (MS1_AD0): no longer R31.1
Changed lines of the file:
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@@
   (junction (at 153.67 78.74) (diameter 0) (color 0 0 0 0)
   )
-  (junction (at 38.1 78.74) (diameter 0) (color 0 0 0 0)
+  (junction (at 38.1 81.28) (diameter 0) (color 0 0 0 0)
   )
   (junction (at 106.68 34.29) (diameter 0) (color 0 0 0 0)
@@
     (stroke (width 0) (type default))
   )
+  (wire (pts (xy 38.1 62.23) (xy 38.1 81.28))
+    (stroke (width 0) (type default))
+  )
   (wire (pts (xy 29.21 78.74) (xy 29.21 82.55))
     (stroke (width 0) (type default))
@@
     (stroke (width 0) (type default))
   )
+  (wire (pts (xy 38.1 81.28) (xy 91.44 81.28))
+    (stroke (width 0) (type default))
+  )
   (wire (pts (xy 106.68 46.99) (xy 106.68 34.29))
     (stroke (width 0) (type default))
@@
     (stroke (width 0) (type default))
   )
-  (wire (pts (xy 38.1 62.23) (xy 38.1 78.74))
-    (stroke (width 0) (type default))
-  )
   (wire (pts (xy 115.57 107.95) (xy 118.11 107.95))
     (stroke (width 0) (type default))
@@
     (stroke (width 0) (type default))
   )
-  (wire (pts (xy 36.83 81.28) (xy 91.44 81.28))
+  (wire (pts (xy 36.83 81.28) (xy 38.1 81.28))
     (stroke (width 0) (type default))
   )
@@
     (stroke (width 0) (type default))
   )
-  (wire (pts (xy 30.48 78.74) (xy 38.1 78.74))
-    (stroke (width 0) (type default))
-  )
   (wire (pts (xy 83.82 63.5) (xy 91.44 63.5))
     (stroke (width 0) (type default))
@@
     (stroke (width 0) (type default))
   )
-  (wire (pts (xy 38.1 78.74) (xy 91.44 78.74))
-    (stroke (width 0) (type default))
-  )
+  (wire (pts (xy 30.48 78.74) (xy 91.44 78.74))
+    (stroke (width 0) (type default))
+  )
