File: Motor_Board_PCB/motor_board_pcb/Motor_Driver_Sheet.kicad_sch (KiCad schematic)
At the start: 25 parts, among them J2 Screw_Terminal_01x04, U4 TMC2209-LA

Commit message: - added footprint labels to schematic symbols
Parts:
- C15, C16, C21, R19, R20, R21, R22, R23, R24, R25, R26, R27, R28, R29, R31, R32, R33: FP (none) -> 0603
- C17, C18, C19, C20, C22: FP (none) -> 0402
Changed lines of the file:
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@@
   )
   (symbol (lib_id "Device:R") (at 22.86 73.66 180) (unit 1)
-    (in_bom yes) (on_board yes) (dnp no) (fields_autoplaced)
+    (in_bom yes) (on_board yes) (dnp no)
     (property "Reference" "R19" (at 25.4 72.39 0)
       (effects (font (size 1.27 1.27)) (justify right))
@@
       (effects (font (size 1.27 1.27)) hide)
     )
+    (property "FP" "0603" (at 26.67 77.47 0)
+      (effects (font (size 1.27 1.27)))
+    )
     (pin "1")
     (pin "2")
@@
   )
   (symbol (lib_id "Device:R") (at 74.93 106.68 180) (unit 1)
-    (in_bom yes) (on_board yes) (dnp no) (fields_autoplaced)
+    (in_bom yes) (on_board yes) (dnp no)
     (property "Reference" "R26" (at 77.47 105.41 0)
       (effects (font (size 1.27 1.27)) (justify right))
@@
       (effects (font (size 1.27 1.27)) hide)
     )
+    (property "FP" "0603" (at 78.74 110.49 0)
+      (effects (font (size 1.27 1.27)))
+    )
     (pin "1")
     (pin "2")
@@
   )
   (symbol (lib_id "Device:R") (at 36.83 86.36 180) (unit 1)
-    (in_bom yes) (on_board yes) (dnp no) (fields_autoplaced)
+    (in_bom yes) (on_board yes) (dnp no)
     (property "Reference" "R21" (at 39.37 85.09 0)
       (effects (font (size 1.27 1.27)) (justify right))
@@
       (effects (font (size 1.27 1.27)) hide)
     )
+    (property "FP" "0603" (at 41.91 90.17 0)
+      (effects (font (size 1.27 1.27)))
+    )
     (pin "1")
     (pin "2")
@@
   )
   (symbol (lib_id "Device:C") (at 76.2 39.37 180) (unit 1)
-    (in_bom yes) (on_board yes) (dnp no) (fields_autoplaced)
+    (in_bom yes) (on_board yes) (dnp no)
     (property "Reference" "C17" (at 80.01 38.1 0)
       (effects (font (size 1.27 1.27)) (justify right))
@@
       (effects (font (size 1.27 1.27)) hide)
     )
+    (property "FP" "0402" (at 82.55 35.56 0)
+      (effects (font (size 1.27 1.27)))
+    )
     (pin "1")
     (pin "2")
@@
   )
   (symbol (lib_id "Device:C") (at 139.7 86.36 180) (unit 1)
-    (in_bom yes) (on_board yes) (dnp no) (fields_autoplaced)
+    (in_bom yes) (on_board yes) (dnp no)
     (property "Reference" "C21" (at 143.51 85.09 0)
       (effects (font (size 1.27 1.27)) (justify right))
@@
     (property "Datasheet" "~" (at 139.7 86.36 0)
       (effects (font (size 1.27 1.27)) hide)
+    )
+    (property "FP" "0603" (at 146.05 90.17 0)
+      (effects (font (size 1.27 1.27)))
     )
     (pin "1")
@@
   )
   (symbol (lib_id "Device:R") (at 38.1 58.42 180) (unit 1)
-    (in_bom yes) (on_board yes) (dnp yes) (fields_autoplaced)
+    (in_bom yes) (on_board yes) (dnp yes)
     (property "Reference" "R31" (at 40.64 57.15 0)
       (effects (font (size 1.27 1.27)) (justify right))
@@
       (effects (font (size 1.27 1.27)) hide)
     )
+    (property "FP" "0603" (at 41.91 62.23 0)
+      (effects (font (size 1.27 1.27)))
+    )
     (pin "1")
     (pin "2")
@@
       (effects (font (size 1.27 1.27)) hide)
     )
+    (property "FP" "0603" (at 69.85 71.12 90)
+      (effects (font (size 1.27 1.27)))
+    )
     (pin "1")
     (pin "2")
@@
   )
   (symbol (lib_id "Device:R") (at 45.72 58.42 180) (unit 1)
-    (in_bom yes) (on_board yes) (dnp yes) (fields_autoplaced)
+    (in_bom yes) (on_board yes) (dnp yes)
     (property "Reference" "R33" (at 48.26 57.15 0)
       (effects (font (size 1.27 1.27)) (justify right))
@@
       (effects (font (size 1.27 1.27)) hide)
     )
+    (property "FP" "0603" (at 49.53 62.23 0)
+      (effects (font (size 1.27 1.27)))
+    )
     (pin "1")
     (pin "2")
@@
       (effects (font (size 1.27 1.27)) hide)
     )
+    (property "FP" "0603" (at 69.85 73.66 90)
+      (effects (font (size 1.27 1.27)))
+    )
     (pin "1")
     (pin "2")
@@
   )
   (symbol (lib_id "Device:C") (at 50.8 39.37 180) (unit 1)
-    (in_bom yes) (on_board yes) (dnp no) (fields_autoplaced)
+    (in_bom yes) (on_board yes) (dnp no)
     (property "Reference" "C15" (at 54.61 38.1 0)
       (effects (font (size 1.27 1.27)) (justify right))
@@
       (effects (font (size 1.27 1.27)) hide)
     )
+    (property "FP" "0603" (at 57.15 35.56 0)
+      (effects (font (size 1.27 1.27)))
+    )
     (pin "1")
     (pin "2")
@@
   )
   (symbol (lib_id "Device:R") (at 148.59 107.95 180) (unit 1)
-    (in_bom yes) (on_board yes) (dnp no) (fields_autoplaced)
+    (in_bom yes) (on_board yes) (dnp no)
     (property "Reference" "R29" (at 151.13 106.68 0)
       (effects (font (size 1.27 1.27)) (justify right))
@@
       (effects (font (size 1.27 1.27)) hide)
     )
+    (property "FP" "0603" (at 153.67 111.76 0)
+      (effects (font (size 1.27 1.27)))
+    )
     (pin "1")
     (pin "2")
@@
   )
   (symbol (lib_id "Device:C") (at 114.3 34.29 270) (unit 1)
-    (in_bom yes) (on_board yes) (dnp no) (fields_autoplaced)
+    (in_bom yes) (on_board yes) (dnp no)
     (property "Reference" "C20" (at 114.3 26.67 90)
       (effects (font (size 1.27 1.27)))
@@
       (effects (font (size 1.27 1.27)) hide)
     )
+    (property "FP" "0402" (at 118.11 33.02 90)
+      (effects (font (size 1.27 1.27)))
+    )
     (pin "1")
     (pin "2")
@@
   )
   (symbol (lib_id "Device:C") (at 63.5 39.37 180) (unit 1)
-    (in_bom yes) (on_board yes) (dnp no) (fields_autoplaced)
+    (in_bom yes) (on_board yes) (dnp no)
     (property "Reference" "C16" (at 67.31 38.1 0)
       (effects (font (size 1.27 1.27)) (justify right))
@@
       (effects (font (size 1.27 1.27)) hide)
     )
+    (property "FP" "0603" (at 69.85 35.56 0)
+      (effects (font (size 1.27 1.27)))
+    )
     (pin "1")
     (pin "2")
@@
   )
   (symbol (lib_id "Device:R") (at 66.04 106.68 180) (unit 1)
-    (in_bom yes) (on_board yes) (dnp no) (fields_autoplaced)
+    (in_bom yes) (on_board yes) (dnp no)
     (property "Reference" "R23" (at 68.58 105.41 0)
       (effects (font (size 1.27 1.27)) (justify right))
@@
       (effects (font (size 1.27 1.27)) hide)
     )
+    (property "FP" "0603" (at 69.85 110.49 0)
+      (effects (font (size 1.27 1.27)))
+    )
     (pin "1")
     (pin "2")
@@
   )
   (symbol (lib_id "Device:R") (at 83.82 106.68 180) (unit 1)
-    (in_bom yes) (on_board yes) (dnp no) (fields_autoplaced)
+    (in_bom yes) (on_board yes) (dnp no)
     (property "Reference" "R27" (at 86.36 105.41 0)
       (effects (font (size 1.27 1.27)) (justify right))
@@
       (effects (font (size 1.27 1.27)) hide)
     )
+    (property "FP" "0603" (at 88.9 110.49 0)
+      (effects (font (size 1.27 1.27)))
+    )
     (pin "1")
     (pin "2")
@@
   )
   (symbol (lib_id "Device:R") (at 29.21 86.36 180) (unit 1)
-    (in_bom yes) (on_board yes) (dnp no) (fields_autoplaced)
+    (in_bom yes) (on_board yes) (dnp no)
     (property "Reference" "R20" (at 31.75 85.09 0)
       (effects (font (size 1.27 1.27)) (justify right))
@@
       (effects (font (size 1.27 1.27)) hide)
     )
+    (property "FP" "0603" (at 25.4 86.36 0)
+      (effects (font (size 1.27 1.27)))
+    )
     (pin "1")
     (pin "2")
@@
   )
   (symbol (lib_id "Device:R") (at 50.8 91.44 180) (unit 1)
-    (in_bom yes) (on_board yes) (dnp no) (fields_autoplaced)
+    (in_bom yes) (on_board yes) (dnp no)
     (property "Reference" "R22" (at 53.34 90.17 0)
       (effects (font (size 1.27 1.27)) (justify right))
@@
       (effects (font (size 1.27 1.27)) hide)
     )
+    (property "FP" "0603" (at 54.61 95.25 0)
+      (effects (font (size 1.27 1.27)))
+    )
     (pin "1")
     (pin "2")
@@
   )
   (symbol (lib_id "Device:R") (at 137.16 107.95 180) (unit 1)
-    (in_bom yes) (on_board yes) (dnp no) (fields_autoplaced)
+    (in_bom yes) (on_board yes) (dnp no)
     (property "Reference" "R28" (at 139.7 106.68 0)
       (effects (font (size 1.27 1.27)) (justify right))
@@
       (effects (font (size 1.27 1.27)) hide)
     )
+    (property "FP" "0603" (at 142.24 111.76 0)
+      (effects (font (size 1.27 1.27)))
+    )
     (pin "1")
     (pin "2")
@@
   )
   (symbol (lib_id "Device:R") (at 30.48 58.42 180) (unit 1)
-    (in_bom yes) (on_board yes) (dnp yes) (fields_autoplaced)
+    (in_bom yes) (on_board yes) (dnp yes)
     (property "Reference" "R32" (at 33.02 57.15 0)
       (effects (font (size 1.27 1.27)) (justify right))
@@
     (property "Datasheet" "~" (at 30.48 58.42 0)
       (effects (font (size 1.27 1.27)) hide)
+    )
+    (property "FP" "0603" (at 34.29 62.23 0)
+      (effects (font (size 1.27 1.27)))
     )
     (pin "1")
@@
   )
   (symbol (lib_id "Device:C") (at 153.67 86.36 0) (unit 1)
-    (in_bom yes) (on_board yes) (dnp no) (fields_autoplaced)
+    (in_bom yes) (on_board yes) (dnp no)
     (property "Reference" "C22" (at 157.48 85.09 0)
       (effects (font (size 1.27 1.27)) (justify left))
@@
       (effects (font (size 1.27 1.27)) hide)
     )
+    (property "FP" "0402" (at 160.02 90.17 0)
+      (effects (font (size 1.27 1.27)))
+    )
     (pin "1")
     (pin "2")
@@
   )
   (symbol (lib_id "Device:C") (at 88.9 39.37 180) (unit 1)
-    (in_bom yes) (on_board yes) (dnp no) (fields_autoplaced)
+    (in_bom yes) (on_board yes) (dnp no)
     (property "Reference" "C19" (at 92.71 38.1 0)
       (effects (font (size 1.27 1.27)) (justify right))
@@
       (effects (font (size 1.27 1.27)) hide)
     )
+    (property "FP" "0402" (at 95.25 35.56 0)
+      (effects (font (size 1.27 1.27)))
+    )
     (pin "1")
     (pin "2")
@@
   )
   (symbol (lib_id "Device:C") (at 83.82 57.15 180) (unit 1)
-    (in_bom yes) (on_board yes) (dnp no) (fields_autoplaced)
+    (in_bom yes) (on_board yes) (dnp no)
     (property "Reference" "C18" (at 87.63 55.88 0)
       (effects (font (size 1.27 1.27)) (justify right))
@@
       (effects (font (size 1.27 1.27)) hide)
     )
-    (pin "1")
+    (property "FP" "0402" (at 81.28 54.61 0)
+      (effects (font (size 1.27 1.27)))
+    )
+    (pin "1")
