File: Motor_Board_PCB/motor_board_pcb/Power_Sheet.kicad_sch (KiCad schematic)
At the start: 16 parts, among them J8 Conn_01x02, U6 AP63205WU-7

Commit message: - added footprint labels to schematic symbols
Parts:
- C23, C26, C28, C29: FP (none) -> 0603
- C27, F1: FP (none) -> 1206
- C30, C32: FP (none) -> 1210
Changed lines of the file:
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@@
   )
   (symbol (lib_id "Device:C") (at 135.89 119.38 180) (unit 1)
-    (in_bom yes) (on_board yes) (dnp no) (fields_autoplaced)
+    (in_bom yes) (on_board yes) (dnp no)
     (property "Reference" "C29" (at 139.7 118.11 0)
       (effects (font (size 1.27 1.27)) (justify right))
@@
     (property "Datasheet" "~" (at 135.89 119.38 0)
       (effects (font (size 1.27 1.27)) hide)
+    )
+    (property "FP" "0603" (at 140.97 123.19 0)
+      (effects (font (size 1.27 1.27)))
     )
     (pin "1")
@@
   )
   (symbol (lib_id "Device:C") (at 39.37 119.38 180) (unit 1)
-    (in_bom yes) (on_board yes) (dnp no) (fields_autoplaced)
+    (in_bom yes) (on_board yes) (dnp no)
     (property "Reference" "C23" (at 43.18 118.11 0)
       (effects (font (size 1.27 1.27)) (justify right))
@@
       (effects (font (size 1.27 1.27)) hide)
     )
+    (property "FP" "0603" (at 45.72 123.19 0)
+      (effects (font (size 1.27 1.27)))
+    )
     (pin "1")
     (pin "2")
@@
   )
   (symbol (lib_id "Device:C") (at 106.68 53.34 180) (unit 1)
-    (in_bom yes) (on_board yes) (dnp no) (fields_autoplaced)
+    (in_bom yes) (on_board yes) (dnp no)
     (property "Reference" "C30" (at 110.49 52.07 0)
       (effects (font (size 1.27 1.27)) (justify right))
@@
       (effects (font (size 1.27 1.27)) hide)
     )
+    (property "FP" "1210" (at 113.03 57.15 0)
+      (effects (font (size 1.27 1.27)))
+    )
     (pin "1")
     (pin "2")
@@
   )
   (symbol (lib_id "Device:C") (at 139.7 53.34 180) (unit 1)
-    (in_bom yes) (on_board yes) (dnp no) (fields_autoplaced)
+    (in_bom yes) (on_board yes) (dnp no)
     (property "Reference" "C32" (at 143.51 52.07 0)
       (effects (font (size 1.27 1.27)) (justify right))
@@
       (effects (font (size 1.27 1.27)) hide)
     )
+    (property "FP" "1210" (at 146.05 57.15 0)
+      (effects (font (size 1.27 1.27)))
+    )
     (pin "1")
     (pin "2")
@@
   )
   (symbol (lib_id "Device:C") (at 81.28 115.57 90) (unit 1)
-    (in_bom yes) (on_board yes) (dnp no) (fields_autoplaced)
+    (in_bom yes) (on_board yes) (dnp no)
     (property "Reference" "C26" (at 81.28 107.95 90)
       (effects (font (size 1.27 1.27)))
@@
     (property "Datasheet" "~" (at 81.28 115.57 0)
       (effects (font (size 1.27 1.27)) hide)
+    )
+    (property "FP" "0603" (at 85.09 116.84 90)
+      (effects (font (size 1.27 1.27)))
     )
     (pin "1")
@@
   )
   (symbol (lib_id "Device:Fuse") (at 63.5 48.26 90) (unit 1)
-    (in_bom yes) (on_board yes) (dnp no) (fields_autoplaced)
+    (in_bom yes) (on_board yes) (dnp no)
     (property "Reference" "F1" (at 63.5 43.18 90)
       (effects (font (size 1.27 1.27)))
@@
       (effects (font (size 1.27 1.27)) hide)
     )
+    (property "FP" "1206" (at 63.5 50.8 90)
+      (effects (font (size 1.27 1.27)))
+    )
     (pin "1")
     (pin "2")
@@
   )
   (symbol (lib_id "Device:C") (at 73.66 53.34 180) (unit 1)
-    (in_bom yes) (on_board yes) (dnp no) (fields_autoplaced)
+    (in_bom yes) (on_board yes) (dnp no)
     (property "Reference" "C27" (at 77.47 52.07 0)
       (effects (font (size 1.27 1.27)) (justify right))
@@
     (property "Datasheet" "~" (at 73.66 53.34 0)
       (effects (font (size 1.27 1.27)) hide)
+    )
+    (property "FP" "1206" (at 80.01 57.15 0)
+      (effects (font (size 1.27 1.27)))
     )
     (pin "1")
@@
   )
   (symbol (lib_id "Device:C") (at 123.19 119.38 180) (unit 1)
-    (in_bom yes) (on_board yes) (dnp no) (fields_autoplaced)
+    (in_bom yes) (on_board yes) (dnp no)
     (property "Reference" "C28" (at 127 118.11 0)
       (effects (font (size 1.27 1.27)) (justify right))
@@
       (effects (font (size 1.27 1.27)) hide)
     )
-    (pin "1")
+    (property "FP" "0603" (at 128.27 123.19 0)
+      (effects (font (size 1.27 1.27)))
+    )
+    (pin "1")
